Commit message: Add files via upload

File: description/gazebo_control.xacro (robot description, xacro)
@@ -6,6 +6,6 @@
             <left_joint>left_wheel_joint</left_joint>
             <right_joint>right_wheel_joint</right_joint>
-            <wheel_separation>0.7</wheel_separation>
-            <wheel_diameter>0.1</wheel_diameter>
+            <wheel_separation>0.8</wheel_separation>
+            <wheel_diameter>0.44</wheel_diameter>
             <!-- Limits -->
             <max_wheel_torque>200</max_wheel_torque>

File: description/lidar.xacro (robot description, xacro)
@@ -4,5 +4,5 @@
         <parent link="chassis"/>
         <child link="laser_frame"/>
-        <origin xyz="0.244 0 0.424" rpy="0 0 0"/>
+        <origin xyz="0.775 0 0.625" rpy="0 0 0"/>
     </joint>
     <link name="laser_frame">
@@ -39,6 +39,6 @@
                     <horizontal>
                         <samples>360</samples>
-                        <min_angle>-3.14</min_angle>
-                        <max_angle>3.14</max_angle>
+                        <min_angle>-2.09</min_angle>
+                        <max_angle>2.09</max_angle>
                     </horizontal>
                 </scan>

File: description/robot.urdf.xacro (robot description, xacro)
@@ -1,12 +1,16 @@
 <?xml version="1.0"?>
-<robot xmlns:xacro="http://www.ros.org/wiki/xacro"  name="learn_one">
+<robot xmlns:xacro="http://www.ros.org/wiki/xacro"  name="robot">
     <xacro:arg name="use_ros2_control" default="true"/>
+    <xacro:arg name="sim_mode" default="false"/>
     <xacro:include filename="robot_core.xacro" />
     <xacro:if value="$(arg use_ros2_control)">
-        <xacro:include filename="ros2_control.xacro"/>
+        <xacro:include filename="ros2_control.xacro" />
     </xacro:if>
     <xacro:unless value="$(arg use_ros2_control)">
-        <xacro:include filename="gazebo_control.xacro"/>
+        <xacro:include filename="gazebo_control.xacro" />
     </xacro:unless>
-    <xacro:include filename="lidar.xacro"/>
+    <xacro:include filename="lidar.xacro" />
+    <!-- <xacro:include filename="camera.xacro" /> -->
+    <!-- <xacro:include filename="depth_camera.xacro" /> -->
+    <xacro:include filename="face.xacro" />
 </robot>

File: description/robot_core.xacro (robot description, xacro)
@@ -36,18 +36,18 @@
     <link name="chassis">
         <visual>
-            <origin xyz="0.3 0 0.15"/>
+            <origin xyz="0.391 0 0.3"/>
             <geometry>
-                <box size="0.6 0.6 0.3"/>
+                <box size="0.782 0.83 0.6"/>
             </geometry>
             <material name="white"/>
         </visual>
         <collision>
-            <origin xyz="0.3 0 0.15"/>
+            <origin xyz="0.391 0 0.3"/>
             <geometry>
-                <box size="0.6 0.6 0.3"/>
+                <box size="0.782 0.83 0.6"/>
             </geometry>
         </collision>
-        <xacro:inertial_box mass="1" x="0.6" y="0.6" z="0.3">
-            <origin xyz="0.3 0 0.15" rpy="0 0 0"/>
+        <xacro:inertial_box mass="1.5" x="0.782" y="0.83" z="0.6">
+            <origin xyz="0.391 0 0.3" rpy="0 0 0"/>
         </xacro:inertial_box>
     </link>
@@ -59,5 +59,5 @@
         <parent link="base_link"/>
         <child link="left_wheel"/>
-        <origin xyz="0 0.35 0" rpy="-${pi/2} 0 0"/>
+        <origin xyz="0.567 0.4 0" rpy="-${pi/2} 0 0"/>
         <axis xyz="0 0 1"/>
     </joint>
@@ -65,5 +65,5 @@
         <visual>
             <geometry>
-                <cylinder radius="0.05" length="0.08"/>
+                <cylinder radius="0.22" length="0.08"/>
             </geometry>
             <material name="blue"/>
@@ -71,8 +71,8 @@
         <collision>
             <geometry>
-                <sphere radius="0.05"/>
+                <sphere radius="0.22"/>
             </geometry>
         </collision>
-        <xacro:inertial_cylinder mass="0.1" length="0.08" radius="0.05">
+        <xacro:inertial_cylinder mass="0.2" length="0.08" radius="0.22">
             <origin xyz="0 0 0" rpy="0 0 0"/>
         </xacro:inertial_cylinder>
@@ -85,5 +85,5 @@
         <parent link="base_link"/>
         <child link="right_wheel"/>
-        <origin xyz="0 -0.35 0" rpy="${pi/2} 0 0"/>
+        <origin xyz="0.567 -0.4 0" rpy="${pi/2} 0 0"/>
         <axis xyz="0 0 -1"/>
     </joint>
@@ -91,5 +91,5 @@
         <visual>
             <geometry>
-                <cylinder radius="0.05" length="0.08"/>
+                <cylinder radius="0.22" length="0.08"/>
             </geometry>
             <material name="blue"/>
@@ -97,8 +97,8 @@
         <collision>
             <geometry>
-                <sphere radius="0.05"/>
+                <sphere radius="0.22"/>
             </geometry>
         </collision>
-        <xacro:inertial_cylinder mass="0.1" length="0.08" radius="0.05">
+        <xacro:inertial_cylinder mass="0.2" length="0.08" radius="0.22">
             <origin xyz="0 0 0" rpy="0 0 0"/>
         </xacro:inertial_cylinder>
@@ -111,10 +111,10 @@
         <parent link="chassis"/>
         <child link="left_caster_wheel"/>
-        <origin xyz="0.5 -0.3 0"/>
+        <origin xyz="0 -0.35 0"/>
     </joint>
     <link name="left_caster_wheel">
         <visual>
             <geometry>
-                <sphere radius="0.05"/>
+                <sphere radius="0.22"/>
             </geometry>
             <material name="black"/>
@@ -122,8 +122,8 @@
         <collision>
             <geometry>
-                <sphere radius="0.05"/>
+                <sphere radius="0.22"/>
             </geometry>
         </collision>
-        <xacro:inertial_sphere mass="0.15" radius="0.05">
+        <xacro:inertial_sphere mass="0.15" radius="0.22">
             <origin xyz="0 0 0" rpy="0 0 0"/>
         </xacro:inertial_sphere>
@@ -138,10 +138,10 @@
         <parent link="chassis"/>
         <child link="right_caster_wheel"/>
-        <origin xyz="0.5 0.3 0"/>
+        <origin xyz="0 0.35 0"/>
     </joint>
     <link name="right_caster_wheel">
         <visual>
             <geometry>
-                <sphere radius="0.05"/>
+                <sphere radius="0.22"/>
             </geometry>
             <material name="black"/>
@@ -149,8 +149,8 @@
         <collision>
             <geometry>
-                <sphere radius="0.05"/>
+                <sphere radius="0.22"/>
             </geometry>
         </collision>
-        <xacro:inertial_sphere mass="0.15" radius="0.05">
+        <xacro:inertial_sphere mass="0.15" radius="0.22">
             <origin xyz="0 0 0" rpy="0 0 0"/>
         </xacro:inertial_sphere>

File: description/ros2_control.xacro (robot description, xacro)
@@ -1,28 +1,61 @@
 <?xml version="1.0"?>
 <robot xmlns:xacro="http://www.ros.org/wiki/xacro">
-    <ros2_control name="GazeboSystem" type="system">
-        <hardware>
-            <plugin>gazebo_ros2_control/GazeboSystem</plugin>
-        </hardware>
-        <joint name="left_wheel_joint">
-            <command_interface name="velocity">
-                <param name="min">-5</param>
-                <param name="max">5</param>
-            </command_interface>
-            <state_interface name="velocity"/>
-            <state_interface name="position"/>
-        </joint>
-        <joint name="right_wheel_joint">
-            <command_interface name="velocity">
-                <param name="min">-10</param>
-                <param name="max">10</param>
-            </command_interface>
-            <state_interface name="velocity"/>
-            <state_interface name="position"/>
-        </joint>
-    </ros2_control>
+    <xacro:unless value="$(arg sim_mode)">
+        <ros2_control name="RealRobot" type="system">
+            <hardware>
+                <plugin>diffdrive_arduino/DiffDriveArduino</plugin>
+                <param name="left_wheel_name">left_wheel_joint</param>
+                <param name="right_wheel_name">right_wheel_joint</param>
+                <param name="loop_rate">30</param>
+                <param name="device">/dev/ttyUSB0</param>
+                <param name="baud_rate">57600</param>
+                <param name="timeout">1000</param>
+                <param name="enc_counts_per_rev">3436</param> //Change this value according to your encoder counts per revolution
+            </hardware>
+            <joint name="left_wheel_joint">
+                <command_interface name="velocity">
+                    <param name="min">-10</param>
+                    <param name="max">10</param>
+                </command_interface>
+                <state_interface name="velocity"/>
+                <state_interface name="position"/>
+            </joint>
+            <joint name="right_wheel_joint">
+                <command_interface name="velocity">
+                    <param name="min">-10</param>
+                    <param name="max">10</param>
+                </command_interface>
+                <state_interface name="velocity"/>
+                <state_interface name="position"/>
+            </joint>
+        </ros2_control>
+    </xacro:unless>
+    <xacro:if value="$(arg sim_mode)">
+        <ros2_control name="GazeboSystem" type="system">
+            <hardware>
+                <plugin>gazebo_ros2_control/GazeboSystem</plugin>
+            </hardware>
+            <joint name="left_wheel_joint">
+                <command_interface name="velocity">
+                    <param name="min">-10</param>
+                    <param name="max">10</param>
+                </command_interface>
+                <state_interface name="velocity"/>
+                <state_interface name="position"/>
+            </joint>
+            <joint name="right_wheel_joint">
+                <command_interface name="velocity">
+                    <param name="min">-10</param>
+                    <param name="max">10</param>
+                </command_interface>
+                <state_interface name="velocity"/>
+                <state_interface name="position"/>
+            </joint>
+        </ros2_control>
+    </xacro:if>
     <gazebo>
         <plugin name="gazebo_ros2_control" filename="libgazebo_ros2_control.so">
             <parameters>$(find learn_one)/config/my_controllers.yaml</parameters>
+            <parameters>$(find learn_one)/config/gaz_ros2_ctl_use_sim.yaml</parameters>
         </plugin>
     </gazebo>
